File: panthera_e73/panthera_e73.kicad_pcb (KiCad board)
At the start: 2 copper layers, 113.5 x 35 mm, 22 parts, among them J1 Conn_01x05_Female, J11 Conn_01x01, J12 Conn_01x04, J2 Conn_01x04, J3 Conn_02x05_Odd_Even, J4 Conn_01x05, J5 Conn_01x05, J6 Conn_02x08_Odd_Even, J7 Conn_02x08_Odd_Even, J8 Conn_01x03, J9 Conn_01x03, U1 E73-2G4M08S1C, U2 MIC5219-3.3YM5, X1 PCB-USB-C

Commit message: e73: fix mislabeled touchpad pins.
Thankfully, the NRF52 can remap its pins arbitrarily, and the interrupt
pin is non-crucial, so no actual change is necessary.
Connections:
- net Net-(J7-Pad5) renamed /TP_INT
- J4 pad 2: /TP_SS -> /TP_SCL
- J4 pad 3: /TP_SCL -> /TP_SDA
- J4 pad 4: /TP_SDA -> /TP_RST

Commit message: e73: fix mislabeled controller number LED pins.
Connections:
- J7 pad 11: /LED_P2_K -> /LED_P3_K
- J7 pad 13: /LED_P3_K -> /LED_P2_K
- J7 pad 15: /LED_P4_K -> /LED_P1_K
- J7 pad 9: /LED_P1_K -> /LED_P4_K
- U1 pad 12: /LED_P4_K -> /LED_P1_K
- U1 pad 13: /LED_P3_K -> /LED_P2_K
- U1 pad 14: /LED_P2_K -> /LED_P3_K
- U1 pad 15: /LED_P1_K -> /LED_P4_K
Routing:
- net /LED_P4_K: track 40.5 -> 50.7 mm
- net /LED_P1_K: track 50.7 -> 40.5 mm
- net /LED_P3_K: track 42.3 -> 49.0 mm
- net /LED_P2_K: track 49.0 -> 42.3 mm
Changed lines of the file:
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@@
       (net 43 /MODE_PS3))
     (pad 14 smd rect (at -2.54 6.33 90) (size 1.524 0.635) (layers F.Cu F.Paste F.Mask)
-      (net 58 /LED_P2_K))
+      (net 57 /LED_P3_K))
     (pad 12 smd rect (at -3.81 6.33 90) (size 1.524 0.635) (layers F.Cu F.Paste F.Mask)
-      (net 56 /LED_P4_K))
+      (net 59 /LED_P1_K))
     (pad 25 smd rect (at 4.45 8.75 90) (size 1.524 0.635) (layers F.Cu F.Paste F.Mask)
       (net 26 "Net-(U1-Pad25)"))
@@
       (net 45 /BUTTON_R3))
     (pad 15 smd rect (at -1.9 8.75 90) (size 1.524 0.635) (layers F.Cu F.Paste F.Mask)
-      (net 59 /LED_P1_K))
+      (net 56 /LED_P4_K))
     (pad 13 smd rect (at -3.17 8.75 90) (size 1.524 0.635) (layers F.Cu F.Paste F.Mask)
-      (net 57 /LED_P3_K))
+      (net 58 /LED_P2_K))
     (pad 11 smd rect (at -4.44 8.75 90) (size 1.524 0.635) (layers F.Cu F.Paste F.Mask)
       (net 39 /BUTTON_PS4))
@@
       (net 1 +3V3))
     (pad 15 thru_hole oval (at 0 17.78 90) (size 1.7 1.7) (drill 1) (layers *.Cu *.Mask)
-      (net 56 /LED_P4_K))
+      (net 59 /LED_P1_K))
     (pad 14 thru_hole oval (at 2.54 15.24 90) (size 1.7 1.7) (drill 1) (layers *.Cu *.Mask)
       (net 39 /BUTTON_PS4))
     (pad 13 thru_hole oval (at 0 15.24 90) (size 1.7 1.7) (drill 1) (layers *.Cu *.Mask)
-      (net 57 /LED_P3_K))
+      (net 58 /LED_P2_K))
     (pad 12 thru_hole oval (at 2.54 12.7 90) (size 1.7 1.7) (drill 1) (layers *.Cu *.Mask)
       (net 40 /MODE_LOCK))
     (pad 11 thru_hole oval (at 0 12.7 90) (size 1.7 1.7) (drill 1) (layers *.Cu *.Mask)
-      (net 58 /LED_P2_K))
+      (net 57 /LED_P3_K))
     (pad 10 thru_hole oval (at 2.54 10.16 90) (size 1.7 1.7) (drill 1) (layers *.Cu *.Mask)
       (net 41 /MODE_LS))
     (pad 9 thru_hole oval (at 0 10.16 90) (size 1.7 1.7) (drill 1) (layers *.Cu *.Mask)
-      (net 59 /LED_P1_K))
+      (net 56 /LED_P4_K))
     (pad 8 thru_hole oval (at 2.54 7.62 90) (size 1.7 1.7) (drill 1) (layers *.Cu *.Mask)
       (net 42 /MODE_RS))
@@
   (segment (start 191.23 104.66) (end 191.23 100.385) (width 0.127) (layer F.Cu) (net 17))
   (segment (start 189.84 106.05) (end 191.23 104.66) (width 0.127) (layer F.Cu) (net 17))
-  (segment (start 126.21 104.94) (end 126.21 108.77) (width 0.127) (layer B.Cu) (net 62))
-  (via (at 126.21 108.77) (size 0.6) (drill 0.3) (layers F.Cu B.Cu) (net 62))
-  (via (at 150.33 108.77) (size 0.6) (drill 0.3) (layers F.Cu B.Cu) (net 62))
-  (segment (start 126.21 108.77) (end 150.33 108.77) (width 0.127) (layer F.Cu) (net 62))
-  (via (at 150.33 99.61) (size 0.6) (drill 0.3) (layers F.Cu B.Cu) (net 62))
-  (segment (start 150.33 108.77) (end 150.33 99.61) (width 0.127) (layer B.Cu) (net 62))
-  (segment (start 150.33 99.61) (end 150.33 100.7825) (width 0.127) (layer F.Cu) (net 62))
   (segment (start 223.600283 92.99221) (end 221.76779 92.99221) (width 0.127) (layer F.Cu) (net 22) (status 10))
   (segment (start 219.44 95.32) (end 219.44 98.4625) (width 0.127) (layer F.Cu) (net 22))
@@
   (segment (start 171.12 95.46) (end 171.12 82.98) (width 0.127) (layer F.Cu) (net 55))
   (segment (start 171.12 82.98) (end 170.78 82.64) (width 0.127) (layer F.Cu) (net 55))
-  (via (at 167.31 99.9) (size 0.6) (drill 0.3) (layers F.Cu B.Cu) (net 56))
-  (segment (start 167.31 95.46) (end 167.31 99.9) (width 0.127) (layer F.Cu) (net 56))
-  (via (at 138.91 106.27) (size 0.6) (drill 0.3) (layers F.Cu B.Cu) (net 56))
-  (segment (start 138.91 104.94) (end 138.91 106.27) (width 0.127) (layer B.Cu) (net 56))
-  (segment (start 138.91 106.27) (end 167.28 106.27) (width 0.127) (layer F.Cu) (net 56))
-  (via (at 167.28 106.27) (size 0.6) (drill 0.3) (layers F.Cu B.Cu) (net 56))
-  (segment (start 167.31 99.9) (end 167.31 106.24) (width 0.127) (layer B.Cu) (net 56))
-  (segment (start 167.31 106.24) (end 167.28 106.27) (width 0.127) (layer B.Cu) (net 56))
-  (via (at 167.95 99.3) (size 0.6) (drill 0.3) (layers F.Cu B.Cu) (net 57))
-  (segment (start 167.95 97.88) (end 167.95 99.3) (width 0.127) (layer F.Cu) (net 57))
-  (segment (start 136.37 104.94) (end 136.37 106.77) (width 0.127) (layer B.Cu) (net 57))
-  (via (at 136.37 106.77) (size 0.6) (drill 0.3) (layers F.Cu B.Cu) (net 57))
-  (via (at 167.95 106.77) (size 0.6) (drill 0.3) (layers F.Cu B.Cu) (net 57))
-  (segment (start 167.95 99.3) (end 167.95 106.77) (width 0.127) (layer B.Cu) (net 57))
-  (segment (start 167.95 106.77) (end 136.37 106.77) (width 0.127) (layer F.Cu) (net 57))
-  (via (at 168.58 99.9) (size 0.6) (drill 0.3) (layers F.Cu B.Cu) (net 58))
-  (segment (start 168.58 95.46) (end 168.58 99.9) (width 0.127) (layer F.Cu) (net 58))
-  (segment (start 168.6 99.92) (end 168.58 99.9) (width 0.127) (layer B.Cu) (net 58))
-  (segment (start 133.83 104.94) (end 133.83 107.27) (width 0.127) (layer B.Cu) (net 58))
-  (via (at 133.83 107.27) (size 0.6) (drill 0.3) (layers F.Cu B.Cu) (net 58))
-  (segment (start 133.83 107.27) (end 133.76 107.27) (width 0.127) (layer F.Cu) (net 58))
-  (via (at 168.58 107.27) (size 0.6) (drill 0.3) (layers F.Cu B.Cu) (net 58))
-  (segment (start 133.83 107.27) (end 168.58 107.27) (width 0.127) (layer F.Cu) (net 58))
-  (segment (start 168.58 99.9) (end 168.58 107.27) (width 0.127) (layer B.Cu) (net 58))
-  (via (at 169.22 99.3) (size 0.6) (drill 0.3) (layers F.Cu B.Cu) (net 59))
-  (segment (start 169.22 97.88) (end 169.22 99.3) (width 0.127) (layer F.Cu) (net 59))
-  (segment (start 169.23 99.31) (end 169.22 99.3) (width 0.127) (layer B.Cu) (net 59))
-  (segment (start 131.29 104.94) (end 131.29 107.77) (width 0.127) (layer B.Cu) (net 59))
-  (segment (start 131.29 107.77) (end 131.29 107.77) (width 0.127) (layer B.Cu) (net 59))
-  (via (at 131.29 107.77) (size 0.6) (drill 0.3) (layers F.Cu B.Cu) (net 59))
-  (via (at 169.22 107.77) (size 0.6) (drill 0.3) (layers F.Cu B.Cu) (net 59))
-  (segment (start 169.22 99.3) (end 169.22 107.77) (width 0.127) (layer B.Cu) (net 59))
-  (segment (start 131.29 107.77) (end 169.22 107.77) (width 0.127) (layer F.Cu) (net 59))
+  (via (at 167.31 99.9) (size 0.6) (drill 0.3) (layers F.Cu B.Cu) (net 59))
+  (segment (start 167.31 95.46) (end 167.31 99.9) (width 0.127) (layer F.Cu) (net 59))
+  (via (at 138.91 106.27) (size 0.6) (drill 0.3) (layers F.Cu B.Cu) (net 59))
+  (segment (start 138.91 104.94) (end 138.91 106.27) (width 0.127) (layer B.Cu) (net 59))
+  (segment (start 138.91 106.27) (end 167.28 106.27) (width 0.127) (layer F.Cu) (net 59))
+  (via (at 167.28 106.27) (size 0.6) (drill 0.3) (layers F.Cu B.Cu) (net 59))
+  (segment (start 167.31 99.9) (end 167.31 106.24) (width 0.127) (layer B.Cu) (net 59))
+  (segment (start 167.31 106.24) (end 167.28 106.27) (width 0.127) (layer B.Cu) (net 59))
+  (via (at 167.95 99.3) (size 0.6) (drill 0.3) (layers F.Cu B.Cu) (net 58))
+  (segment (start 167.95 97.88) (end 167.95 99.3) (width 0.127) (layer F.Cu) (net 58))
+  (segment (start 136.37 104.94) (end 136.37 106.77) (width 0.127) (layer B.Cu) (net 58))
+  (via (at 136.37 106.77) (size 0.6) (drill 0.3) (layers F.Cu B.Cu) (net 58))
+  (via (at 167.95 106.77) (size 0.6) (drill 0.3) (layers F.Cu B.Cu) (net 58))
+  (segment (start 167.95 99.3) (end 167.95 106.77) (width 0.127) (layer B.Cu) (net 58))
+  (segment (start 167.95 106.77) (end 136.37 106.77) (width 0.127) (layer F.Cu) (net 58))
+  (via (at 168.58 99.9) (size 0.6) (drill 0.3) (layers F.Cu B.Cu) (net 57))
+  (segment (start 168.58 95.46) (end 168.58 99.9) (width 0.127) (layer F.Cu) (net 57))
+  (segment (start 168.6 99.92) (end 168.58 99.9) (width 0.127) (layer B.Cu) (net 57))
+  (segment (start 133.83 104.94) (end 133.83 107.27) (width 0.127) (layer B.Cu) (net 57))
+  (via (at 133.83 107.27) (size 0.6) (drill 0.3) (layers F.Cu B.Cu) (net 57))
+  (segment (start 133.83 107.27) (end 133.76 107.27) (width 0.127) (layer F.Cu) (net 57))
+  (via (at 168.58 107.27) (size 0.6) (drill 0.3) (layers F.Cu B.Cu) (net 57))
+  (segment (start 133.83 107.27) (end 168.58 107.27) (width 0.127) (layer F.Cu) (net 57))
+  (segment (start 168.58 99.9) (end 168.58 107.27) (width 0.127) (layer B.Cu) (net 57))
+  (via (at 169.22 99.3) (size 0.6) (drill 0.3) (layers F.Cu B.Cu) (net 56))
+  (segment (start 169.22 97.88) (end 169.22 99.3) (width 0.127) (layer F.Cu) (net 56))
+  (segment (start 169.23 99.31) (end 169.22 99.3) (width 0.127) (layer B.Cu) (net 56))
+  (segment (start 131.29 104.94) (end 131.29 107.77) (width 0.127) (layer B.Cu) (net 56))
+  (segment (start 131.29 107.77) (end 131.29 107.77) (width 0.127) (layer B.Cu) (net 56))
+  (via (at 131.29 107.77) (size 0.6) (drill 0.3) (layers F.Cu B.Cu) (net 56))
+  (via (at 169.22 107.77) (size 0.6) (drill 0.3) (layers F.Cu B.Cu) (net 56))
+  (segment (start 169.22 99.3) (end 169.22 107.77) (width 0.127) (layer B.Cu) (net 56))
+  (segment (start 131.29 107.77) (end 169.22 107.77) (width 0.127) (layer F.Cu) (net 56))
   (segment (start 223.600283 91.49221) (end 221.35221 91.49221) (width 0.127) (layer B.Cu) (net 60) (status 10))
   (segment (start 221.35221 91.49221) (end 221.03 91.17) (width 0.127) (layer B.Cu) (net 60))
@@
   (segment (start 218.85 89.1275) (end 219.44 88.5375) (width 0.127) (layer F.Cu) (net 60))
   (segment (start 218.85 91.17) (end 218.85 89.1275) (width 0.127) (layer F.Cu) (net 60))
+  (segment (start 126.21 104.94) (end 126.21 108.77) (width 0.127) (layer B.Cu) (net 62))
+  (via (at 126.21 108.77) (size 0.6) (drill 0.3) (layers F.Cu B.Cu) (net 62))
+  (via (at 150.33 108.77) (size 0.6) (drill 0.3) (layers F.Cu B.Cu) (net 62))
+  (segment (start 126.21 108.77) (end 150.33 108.77) (width 0.127) (layer F.Cu) (net 62))
+  (via (at 150.33 99.61) (size 0.6) (drill 0.3) (layers F.Cu B.Cu) (net 62))
+  (segment (start 150.33 108.77) (end 150.33 99.61) (width 0.127) (layer B.Cu) (net 62))
+  (segment (start 150.33 99.61) (end 150.33 100.7825) (width 0.127) (layer F.Cu) (net 62))
   (zone (net 2) (net_name GND) (layer F.Cu) (hatch edge 0.508)
     (connect_pads (clearance 0.1524))
